File: 4_Schematics and Boards Layout/4_6_Schematics/MainBoard/RADAR_Main_Board.brd (EAGLE design)
At the start: 260 x 300 mm, 776 parts, among them J1 142-0731-211, J18 142-0731-211, J19 CJT-T-P-HH-ST-TH1, J20 142-0731-211, J21 CJT-T-P-HH-ST-TH1, J22 142-0731-211, J23 142-0731-211, J24 142-0731-211, J25 142-0731-211, J26 142-0731-211, J27 142-0731-211, J28 142-0731-211, J29 142-0731-211, J30 142-0731-211, J31 142-0731-211, J32 142-0731-211, J33 142-0731-211, J34 142-0731-211, J35 142-0731-211, J36 142-0731-211, J37 142-0731-211, J38 142-0731-211, J39 142-0731-211, J40 142-0731-211, J41 142-0731-211, J42 142-0731-211, J43 142-0731-211, J44 142-0731-211, J45 142-0731-211, J46 142-0731-211, J47 142-0731-211, J48 142-0731-211, J49 142-0731-211, J50 142-0731-211, J51 142-0731-211, J52 142-0731-211, J53 142-0731-211, J54 142-0731-211, J55 142-0731-211, U1 AD9484BCPZ-500, U10 ADS7830IPWR, U11 INA241A3IDGKRDGK0008A-MFG, U13 LTC5552IUDBTRMPBF, U14 SZMMSZ5232BT1G, U15 SZMMSZ5232BT1G, U16 EP4RKU+, U17 SZMMSZ5232BT1G, U2 STM32F746ZGT7, U3 AD9708AR, U37 SZMMSZ5232BT1G, U38 SZMMSZ5232BT1G, U39 SZMMSZ5232BT1G, U4 AD8352ACPZ-R7, U40 SZMMSZ5232BT1G, U41 SZMMSZ5232BT1G, U42 XC7A50T-2FTG256I, U43 SZMMSZ5232BT1G, U44 SZMMSZ5232BT1G, U45 SZMMSZ5232BT1G, U46 SZMMSZ5232BT1G, U47 SZMMSZ5232BT1G, U48 SZMMSZ5232BT1G, U49 SZMMSZ5232BT1G, U5 LTC5552IUDBTRMPBF, U50 SZMMSZ5232BT1G, U51 SZMMSZ5232BT1G, U52 SZMMSZ5232BT1G, U53 SZMMSZ5232BT1G, U54 SZMMSZ5232BT1G, U55 SZMMSZ5232BT1G, U56 SZMMSZ5232BT1G, U57 SZMMSZ5232BT1G, U58 SZMMSZ5232BT1G, U59 SZMMSZ5232BT1G, U6 FT601Q-B-T, U60 SZMMSZ5232BT1G, U61 SZMMSZ5232BT1G, U62 SZMMSZ5232BT1G, U63 SZMMSZ5232BT1G, U64 SZMMSZ5232BT1G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

Commit message: Add files via upload
Parts:
- added C187: 4.7uF 35V, SparkFun-Capacitors:EIA3528
- added C188, C189, C190, C192, C193, C194, C195: 0.1uF, eagle-ltspice:C0201
- added C191: 3.3uF, eagle-ltspice:C0201
- added IC1: AT93C46A-10SQ-2.7, atmel:SOIC8
- added L20: BLM15HB121SN1, inductors:0402
- added X2: MINI-USB-32005-201, con-cypressindustries:32005-201
- added Y1: ECS-120-10-36B2-JTN-TR, SparkFun-Clocks:CRYSTAL-SMD-2X2.5MM
- C159: value 22µF -> 0.1uF; device rcl:C1206 -> eagle-ltspice:C0201
- C184: value 10µF -> 12pF; device rcl:C0805 -> eagle-ltspice:C0201
- C185: value 100nF -> 12pF; device rcl:C0402 -> eagle-ltspice:C0201
- C186: value 1nF -> 4.7uF 35V; device rcl:C0402 -> SparkFun-Capacitors:EIA3528
- L19: value (none) -> BLM15HB121SN1; device rcl:L5650M -> inductors:0402
- R145, R83, R84: value 33R -> 10k
- R146: value 33R -> 2.2k
- R60: value 33R -> 1k2_1%
- R61: value 33R -> 1k
- U6: value FT601Q-B-T -> FT2232HQ; device My_Library_RADAR:QFN76_FTD -> My_Library_RADAR:64QFN_FT2232HQ_FTD
- moved C159 353.1 mm to (176.9, 237.1), turned to 180 degrees
- moved C185 343.3 mm to (172.1, 222.5), turned to 90 degrees
- moved R146 338.1 mm to (180.5, 229.9), turned to 270 degrees
- moved C184 337.8 mm to (170.9, 225.8), turned to 90 degrees
- moved C186 332.9 mm to (167.6, 216.7), turned to 90 degrees
- moved R145 328.2 mm to (174.2, 226.9), turned to 180 degrees
- moved L19 327.0 mm to (161.0, 222.9), turned to 180 degrees
- moved R84 326.8 mm to (173.7, 230.3), turned to 180 degrees
- moved R83 325.7 mm to (181.2, 228.9)
- moved R61 307.5 mm to (172.9, 217.3)
- moved R60 307.4 mm to (173.8, 221.4), turned to 180 degrees
- moved U6 152.3 mm to (179.2, 220.1)
- moved C102 143.8 mm to (282.8, 227.9)
- moved C104 143.8 mm to (303.1, 238.3)
- moved C106 143.8 mm to (358.9, 227.9)
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Connections:
- removed net +3V3_FT: C184.1, C185.1, C186.1, L19.2
- removed net AVDD: U6.2
- removed net VBUS: U6.37
- removed net VCC33: U6.38
- removed net VCC33_2: U6.20
- removed net VCC33_3: U6.24
- removed net VCCIO: U6.68
- removed net VCCIO_2: U6.14
- removed net VCCIO_3: U6.49
- removed net VCCIO_4: U6.59
- removed net VDDA: U6.28
- new net FT2232_USB_D_N: U6.7, X2.2
- new net FT2232_USB_D_P: U6.8, X2.3
- new net FT_+1V8: C191.2, U6.12, U6.37, U6.49, U6.64
- new net FT_CLKOUT: U42.C4, U6.32
- new net FT_D0: U42.K1, U6.16
- new net FT_D1: U42.J3, U6.17
- new net FT_D2: U42.H3, U6.18
- new net FT_D3: U42.G4, U6.19
- new net FT_D4: U42.F2, U6.21
- new net FT_D5: U42.D1, U6.22
- new net FT_D6: U42.C3, U6.23
- new net FT_D7: U42.C1, U6.24
- new net FT_OE#: U42.B7, U6.33
- new net FT_RD#: U42.A3, U6.28
- new net FT_RESET#: R61.2, U6.14
- new net FT_RXF#: U42.A2, U6.26
- new net FT_SIWUA: U42.A5, U6.30
- new net FT_TXE#: U42.B2, U6.27
- new net FT_WR#: U42.A4, U6.29
- new net N$117: R60.1, U6.6
- new net N$118: C184.1, U6.2, Y1.P1
- new net N$119: C185.1, U6.3, Y1.P3
- new net N$120: C186.A, C188.2, L20.1, U6.9
- new net N$121: C187.A, C189.1, L19.1, U6.4
- new net N$122: IC1.1, R145.1, U6.63
- new net N$123: IC1.2, R84.1, U6.62
- new net N$124: IC1.3, R146.1, U6.61
- new net N$90: IC1.4, R146.2, R83.1
- net +3V3_FPGA: now also C159.2, C190.2, C192.2, C193.2, C194.2, C195.2, IC1.8, L19.2, L20.2, R145.2, R61.1, R83.2, R84.2, U6.20, U6.31, U6.42, U6.50, U6.56; no longer C159.1, L19.1
- net GND: now also C159.1, C186.C, C187.C, C188.1, C189.2, C190.1, C191.1, C192.1, C193.1, C194.1, C195.1, IC1.5, R60.2, U6.1, U6.10, U6.11, U6.13, U6.15, U6.25, U6.35, U6.47, U6.5, U6.51, U6.65, X2.4, X2.5; no longer C159.2, C186.2
Routing:
- net +3V3_FPGA: track 75.3 -> 375.5 mm, vias 38 -> 50
- net STM32_MISO_1V8: track 615.9 -> 568.8 mm, vias 6 -> 7
- net FT_D0: track 0.00 -> 31.7 mm
- net FT_D1: track 0.00 -> 30.4 mm
- net FT_D2: track 0.00 -> 28.3 mm
- net GND: track 1032.4 -> 1060.6 mm, vias 2183 -> 2711
- net FT_D3: track 0.00 -> 26.8 mm
- net FT2232_USB_D_N: track 0.00 -> 23.5 mm
- net FT2232_USB_D_P: track 0.00 -> 23.5 mm
- net FT_D4: track 0.00 -> 22.7 mm
- net M3S_VCTRL: track 659.7 -> 679.1 mm
- net FT_D6: track 0.00 -> 17.7 mm
- net FT_D5: track 0.00 -> 17.6 mm
- net FT_CLKOUT: track 0.00 -> 17.5 mm
- net FT_OE#: track 0.00 -> 15.9 mm
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- added copper zone on layer 3, net FT_+1V8
Other:
- board text added: "+ -"
- board text added: "+1V0_FPGA"
- board text added: "+1V8_CLOCK"
- board text added: "+1V8_FPGA"
- board text added: "+3V3"
- board text added: "+3V3_ADAR12"
- board text added: "+3V3_ADAR34"
- board text added: "+3V3_ADTR"
- board text added: "+3V3_AN"
- board text added: "+3V3_AN4_F"
- board text added: "+3V3_FPGA"
- board text added: "+3V3_VDD_SW"
- board text added: "+3V4"
- board text added: "+5V0_0"
- board text added: "+5V0_PA_1"
- board text added: "+5V0_PA_2"
- board text added: "+5V0_PA_3"
- board text added: "+5V5_PA"
- board text added: "- +"
- board text added: "-3V3_SW"
- board text added: "-3V4"
- board text added: "-5V0_ADAR12"
- board text added: "-5V0_ADAR34"
- board text added: "-5V5_PA"
- board text added: "AD9523_CS"
- board text added: "AD9523_EEPROM_SEL"
- board text added: "AD9523_PD"
- board text added: "AD9523_REF_SEL"
- board text added: "AD9523_RESET"
- board text added: "AD9523_STATUS0"
- board text added: "AD9523_STATUS1"
- board text added: "AD9523_SYNC"
- board text added: "ADC_CLK_IN"
- board text added: "AERIS-10"
- board text added: "CHAN1"
- board text added: "CHAN10"
- board text added: "CHAN11"
- board text added: "CHAN12"
- board text added: "CHAN13"
- board text added: "CHAN14"
- board text added: "CHAN15"
- board text added: "CHAN16"
- board text added: "CHAN2"
- board text added: "CHAN3"
- board text added: "CHAN4"
- board text added: "CHAN5"
- board text added: "CHAN6"
- board text added: "CHAN7"
- board text added: "CHAN8"
- board text added: "CHAN9"
- board text added: "DAC_CLOCK"
- board text added: "FPGA_ADC_CLOCK"
- board text added: "FPGA_CLOCK_TEST"
- board text added: "FPGA_DAC_CLOCK"
- board text added: "FPGA_SYS_CLOCK"
- board text added: "GND"
- board text added: "JP10"
- board text added: "JP13"
- board text added: "JP18"
- board text added: "JP2"
- board text added: "JP4"
- board text added: "JP7"
- board text added: "JP8"
- board text added: "JP9"
- board text added: "MAIN BOARD"
- board text added: "RX_LO"
- board text added: "STEPPER_CLK+"
- board text added: "STM32_MISO4"
- board text added: "STM32_MOSI4"
- board text added: "STM32_SCLK4"
- board text added: "SV1"
- board text added: "TX_LO"
- board text added: "T°C_1"
- board text added: "T°C_8"
- board text added: "VG_1"
- board text added: "VG_10"
- board text added: "VG_11"
- board text added: "VG_12"
- board text added: "VG_13"
- board text added: "VG_14"
- board text added: "VG_15"
- board text added: "VG_16"
- board text added: "VG_2"
- board text added: "VG_3"
- board text added: "VG_4"
- board text added: "VG_5"
- board text added: "VG_6"
- board text added: "VG_7"
- board text added: "VG_8"
- board text added: "VG_9"
- board text added: "VOLTAGE SEQUENCING"
